File: v1.2/A2PICO2.v1.2.kicad_pcb (KiCad board)
At the start: 4 copper layers, 65.5 x 37.7 mm, 115 parts, among them J1 SolderJumper-2_P1.3mm_Bridged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, SW1 YTS-A016-X, SW2 YTS-A016-X, U1 RP2354B, U2 SN74LVC1G11DBVR, U3 ME6211, X1 Crystal_SMD_Abracon_ABM8AIG-4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

Commit message: Add files via upload
Routing:
- net ~{IRQ}: track 75.1 -> 71.5 mm
- net PHI0: track 48.8 -> 45.3 mm
- net ~{IOSel}: track 43.9 -> 45.3 mm, vias 0 -> 2
- net GND: vias 61 -> 60
Changed lines of the file:
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@@
 	)
 	(via
+		(at 127.4064 107.2134)
+		(size 0.6)
+		(drill 0.3)
+		(layers "F.Cu" "B.Cu")
+		(free yes)
+		(net 2)
+	)
+	(via
 		(at 144.8308 110.2868)
 		(size 0.6)
@@
 	)
 	(via
-		(at 124.3584 104.2416)
-		(size 0.6)
-		(drill 0.3)
-		(layers "F.Cu" "B.Cu")
-		(free yes)
-		(net 2)
-	)
-	(via
 		(at 146.558138 107.7024)
 		(size 0.6)
@@
 	)
 	(via
-		(at 122.3772 107.4928)
-		(size 0.6)
-		(drill 0.3)
-		(layers "F.Cu" "B.Cu")
-		(free yes)
-		(net 2)
-	)
-	(via
 		(at 135.99295 88.509754)
 		(size 0.6)
@@
 	)
 	(segment
-		(start 125.1458 106.426)
-		(end 125.1458 102.927338)
+		(start 120.660144 110.236)
+		(end 120.660144 110.225856)
 		(width 0.15)
 		(layer "B.Cu")
@@
 	)
 	(segment
-		(start 132.320282 95.752856)
-		(end 132.320282 95.277354)
+		(start 125.1458 105.7402)
+		(end 125.1458 102.927338)
 		(width 0.15)
 		(layer "B.Cu")
@@
 	)
 	(segment
-		(start 121.3358 110.236)
-		(end 125.1458 106.426)
+		(start 132.320282 95.752856)
+		(end 132.320282 95.277354)
 		(width 0.15)
 		(layer "B.Cu")
@@
 	)
 	(segment
-		(start 120.660144 110.236)
-		(end 121.3358 110.236)
+		(start 125.1458 102.927338)
+		(end 132.320282 95.752856)
 		(width 0.15)
 		(layer "B.Cu")
@@
 	)
 	(segment
-		(start 125.1458 102.927338)
-		(end 132.320282 95.752856)
+		(start 120.660144 110.225856)
+		(end 125.1458 105.7402)
 		(width 0.15)
 		(layer "B.Cu")
@@
 	)
 	(segment
-		(start 131.670282 93.283158)
-		(end 132.093686 92.859754)
+		(start 122.323468 106.880268)
+		(end 124.6632 109.22)
 		(width 0.15)
 		(layer "F.Cu")
@@
 	)
 	(segment
-		(start 131.845282 94.481882)
-		(end 131.670282 94.306882)
+		(start 131.670282 93.283158)
+		(end 132.093686 92.859754)
 		(width 0.15)
 		(layer "F.Cu")
@@
 	)
 	(segment
-		(start 121.4882 109.22)
-		(end 141.077781 109.22)
+		(start 131.845282 94.481882)
+		(end 131.670282 94.306882)
 		(width 0.15)
 		(layer "F.Cu")
@@
 	)
 	(segment
-		(start 141.788981 109.9312)
-		(end 142.6718 109.9312)
+		(start 141.077781 109.22)
+		(end 141.788981 109.9312)
 		(width 0.15)
 		(layer "F.Cu")
@@
 	)
 	(segment
-		(start 141.077781 109.22)
-		(end 141.788981 109.9312)
+		(start 124.6632 109.22)
+		(end 141.077781 109.22)
 		(width 0.15)
 		(layer "F.Cu")
@@
 	)
 	(segment
-		(start 121.158 109.5502)
-		(end 121.4882 109.22)
+		(start 141.788981 109.9312)
+		(end 142.6718 109.9312)
 		(width 0.15)
 		(layer "F.Cu")
@@
 	)
 	(via
-		(at 121.158 109.5502)
+		(at 122.323468 106.880268)
 		(size 0.6)
 		(drill 0.3)
@@
 	)
 	(segment
-		(start 131.845282 95.474106)
-		(end 121.158 106.161388)
+		(start 122.936 106.267736)
+		(end 122.936 104.383388)
 		(width 0.15)
 		(layer "B.Cu")
@@
 	)
 	(segment
+		(start 122.936 104.383388)
+		(end 131.845282 95.474106)
+		(width 0.15)
+		(layer "B.Cu")
+		(net 34)
+	)
+	(segment
 		(start 142.6718 109.9312)
 		(end 143.520144 110.779544)
@@
 	)
 	(segment
-		(start 121.158 106.161388)
-		(end 121.158 109.5502)
+		(start 131.845282 95.474106)
+		(end 131.845282 94.827354)
 		(width 0.15)
 		(layer "B.Cu")
@@
 	)
 	(segment
-		(start 131.845282 94.827354)
-		(end 131.845282 95.474106)
+		(start 122.323468 106.880268)
+		(end 122.936 106.267736)
 		(width 0.15)
 		(layer "B.Cu")
@@
 	)
 	(segment
-		(start 118.120144 114.6847)
-		(end 118.120144 110.987856)
-		(width 0.2)
-		(layer "F.Cu")
-		(net 35)
-	)
-	(segment
-		(start 153.7106 104.1908)
-		(end 153.7106 104.5058)
+		(start 125.6538 108.2548)
+		(end 123.6726 106.2736)
 		(width 0.15)
 		(layer "F.Cu")
@@
 	)
 	(segment
-		(start 120.4214 108.2548)
-		(end 119.9896 108.6866)
+		(start 153.0604 107.5436)
+		(end 152.3492 108.2548)
 		(width 0.15)
 		(layer "F.Cu")
@@
 	)
 	(segment
-		(start 119.9896 109.1184)
-		(end 119.1886 109.9194)
+		(start 153.0604 105.156)
+		(end 153.0604 107.5436)
 		(width 0.15)
 		(layer "F.Cu")
@@
 	)
 	(segment
-		(start 153.0604 105.156)
-		(end 153.0604 107.5436)
+		(start 153.7106 104.5058)
+		(end 153.0604 105.156)
 		(width 0.15)
 		(layer "F.Cu")
@@
 	(segment
 		(start 118.120144 110.987856)
-		(end 119.1886 109.9194)
+		(end 118.6561 110.4519)
 		(width 0.2)
 		(layer "F.Cu")
@@
 	)
 	(segment
-		(start 153.7106 104.5058)
-		(end 153.0604 105.156)
+		(start 153.7106 104.1908)
+		(end 153.7106 104.5058)
 		(width 0.15)
 		(layer "F.Cu")
@@
 	)
 	(segment
-		(start 119.9896 108.6866)
-		(end 119.9896 109.1184)
-		(width 0.15)
+		(start 118.120144 114.6847)
+		(end 118.120144 110.987856)
+		(width 0.2)
 		(layer "F.Cu")
 		(net 35)
 	)
 	(segment
-		(start 153.0604 107.5436)
-		(end 152.3492 108.2548)
+		(start 152.3492 108.2548)
+		(end 125.6538 108.2548)
 		(width 0.15)
 		(layer "F.Cu")
 		(net 35)
 	)
+	(via
+		(at 123.6726 106.2736)
+		(size 0.6)
+		(drill 0.3)
+		(layers "F.Cu" "B.Cu")
+		(net 35)
+	)
+	(via
+		(at 118.6561 110.4519)
+		(size 0.6)
+		(drill 0.3)
+		(layers "F.Cu" "B.Cu")
+		(net 35)
+	)
 	(segment
-		(start 152.3492 108.2548)
-		(end 120.4214 108.2548)
+		(start 119.4943 110.4519)
+		(end 123.6726 106.2736)
 		(width 0.15)
-		(layer "F.Cu")
+		(layer "B.Cu")
+		(net 35)
+	)
+	(segment
+		(start 118.6561 110.4519)
+		(end 119.4943 110.4519)
+		(width 0.15)
+		(layer "B.Cu")
 		(net 35)
 	)
@@
 		(start 121.3358 110.6678)
 		(end 121.666 110.6678)
-		(width 0.15)
+		(width 0.2)
 		(layer "B.Cu")
 		(net 37)
@@
 	)
 	(segment
-		(start 120.6246 108.8644)
-		(end 120.7008 108.7882)
+		(start 131.370282 93.107422)
+		(end 132.01795 92.459754)
 		(width 0.15)
 		(layer "F.Cu")
@@
 	)
 	(segment
-		(start 131.370282 93.107422)
-		(end 132.01795 92.459754)
+		(start 131.370282 95.277354)
+		(end 131.370282 93.107422)
 		(width 0.15)
 		(layer "F.Cu")
@@
 	)
 	(segment
-		(start 120.7008 108.7882)
+		(start 125.1712 108.7882)
 		(end 141.1732 108.7882)
 		(width 0.15)
@@
 	)
 	(segment
-		(start 141.1732 108.7882)
-		(end 141.6898 109.3048)
+		(start 164.685 109.3048)
+		(end 165.227 108.7628)
 		(width 0.15)
 		(layer "F.Cu")
@@
 	)
 	(segment
-		(start 131.370282 95.277354)
-		(end 131.370282 93.107422)
+		(start 121.541932 105.158932)
+		(end 125.1712 108.7882)
 		(width 0.15)
 		(layer "F.Cu")
@@
 	)
 	(segment
-		(start 164.685 109.3048)
-		(end 165.227 108.7628)
+		(start 132.01795 92.459754)
+		(end 132.46795 92.459754)
 		(width 0.15)
 		(layer "F.Cu")
@@
 	)
 	(segment
-		(start 132.01795 92.459754)
-		(end 132.46795 92.459754)
+		(start 141.1732 108.7882)
+		(end 141.6898 109.3048)
 		(width 0.15)
 		(layer "F.Cu")
@@
 	)
 	(via
-		(at 120.6246 108.8644)
+		(at 121.541932 105.158932)
 		(size 0.6)
 		(drill 0.3)
@@
 	)
 	(segment
-		(start 120.6246 108.8644)
-		(end 120.65 108.839)
-		(width 0.15)
-		(layer "B.Cu")
-		(net 44)
-	)
-	(segment
-		(start 120.65 108.839)
-		(end 120.65 105.997636)
+		(start 121.541932 105.105704)
+		(end 131.370282 95.277354)
 		(width 0.15)
 		(layer "B.Cu")
@@
 	)
 	(segment
-		(start 120.65 105.997636)
-		(end 131.370282 95.277354)
+		(start 121.541932 105.158932)
+		(end 121.541932 105.105704)
 		(width 0.15)
 		(layer "B.Cu")

Commit message: Add files via upload
Parts:
- removed REF**: OSHW-Logo2_7.3x6mm_SilkScreen, Symbol:OSHW-Logo2_7.3x6mm_SilkScreen
- H2: value PinHeader_1x05_P2.54mm_Vertical -> PinHeader_1x05_P2.54mm_Horizontal; footprint Connector_PinHeader_2.54mm:PinHeader_1x05_P2.54mm_Vertical -> Connector_PinHeader_2.54mm:PinHeader_1x05_P2.54mm_Horizontal
Other:
- board text removed: "A2PICO2"

Commit message: Add files via upload
Parts:
- moved H2 2.11 mm to (119.9, 108.8)
Routing:
- net UART_CTS: track 32.2 -> 30.0 mm
- net UART_Rx: track 33.3 -> 31.2 mm
- net UART_RTS: track 33.0 -> 30.9 mm
- net UART_Tx: track 35.6 -> 33.5 mm
- net ~{IOSel}: track 45.3 -> 47.0 mm
- net ~{IRQ}: track 71.5 -> 70.7 mm
- net GND: vias 60 -> 66

Commit message: Add files via upload
Parts:
- H3: value microSD_HC_Molex_104031-0811 -> microSD_Shou_Han; footprint Connector_Card:microSD_HC_Molex_104031-0811 -> Connector_Card:microSD_HC_Hirose_DM3AT-SF-PEJM5
- moved C19 15.5 mm to (166.7, 98.3), turned to 0 degrees
- moved H3 1.14 mm to (164.5, 88.4), turned to 180 degrees
Connections:
- H3 pad 10: Detect -> GND
- H3 pad 9: GND -> Detect
Routing:
- net CMD_: track 24.7 -> 12.6 mm
- net CLK_: track 24.7 -> 13.8 mm
- net DAT2_: track 23.0 -> 13.4 mm
- net DAT3_: track 24.6 -> 15.5 mm
- net Detect: track 37.5 -> 44.6 mm
- net +3V3: track 73.0 -> 66.9 mm
- net DAT0_: track 24.1 -> 18.1 mm
- net DAT1_: track 24.9 -> 20.2 mm
- net GND: track 60.6 -> 62.1 mm, vias 66 -> 69
