File: v1.2/A2PICO2.v1.2.kicad_pcb (KiCad board)
At the start: 4 copper layers, 65.5 x 37.7 mm, 114 parts, among them J1 SolderJumper-2_P1.3mm_Bridged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, SW1 YTS-A016-X, SW2 YTS-A016-X, U1 RP2354B, U2 SN74LVC1G11DBVR, U3 ME6211, X1 Crystal_SMD_Abracon_ABM8AIG-4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

Commit message: Add files via upload
Parts:
- removed C24: 100uF, Capacitor_SMD:C_1206_3216Metric
Changed lines of the file:
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@@
 		(tags "A40-00119-A52-12 is fully compatible to GCT's USB4105-GF-A. See: https://gct.co/connector/usb4105")
 		(property "Reference" "H1"
-			(at -4.536618 -6.326518 180)
+			(at -0.752018 6.170282 180)
 			(layer "F.SilkS")
 			(effects
@@
 		(tags "Micro SD")
 		(property "Reference" "H3"
-			(at -10.1854 -1.7018 0)
+			(at 9.4996 6.4516 0)
 			(layer "F.SilkS")
 			(effects
@@
 			(offset
 				(xyz 0 0 0)
-			)
-			(scale
-				(xyz 1 1 1)
-			)
-			(rotate
-				(xyz 0 0 0)
-			)
-		)
-	)
-	(footprint "Capacitor_SMD:C_1206_3216Metric"
-		(layer "F.Cu")
-		(at 179.0446 106.426 90)
-		(descr "Capacitor SMD 1206 (3216 Metric), square (rectangular) end terminal, IPC_7351 nominal, (Body size source: IPC-SM-782 page 76, https://www.pcb-3d.com/wordpress/wp-content/uploads/ipc-sm-782a_amendment_1_and_2.pdf), generated with kicad-footprint-generator")
-		(tags "capacitor")
-		(property "Reference" "C24"
-			(at -2.6162 0.0788 0)
-			(layer "F.SilkS")
-			(effects
-				(font
-					(size 0.5 0.5)
-					(thickness 0.1)
-					(bold yes)
-				)
-			)
-		)
-		(property "Value" "100uF"
-			(at 0 1.85 90)
-			(layer "F.Fab")
-			(hide yes)
-			(effects
-				(font
-					(size 1 1)
-					(thickness 0.15)
-				)
-			)
-		)
-		(property "Footprint" "Capacitor_SMD:C_1206_3216Metric"
-			(at 0 0 90)
-			(unlocked yes)
-			(layer "F.Fab")
-			(hide yes)
-			(effects
-				(font
-					(size 1.27 1.27)
-					(thickness 0.15)
-				)
-			)
-		)
-		(property "Datasheet" ""
-			(at 0 0 90)
-			(unlocked yes)
-			(layer "F.Fab")
-			(hide yes)
-			(effects
-				(font
-					(size 1.27 1.27)
-					(thickness 0.15)
-				)
-			)
-		)
-		(property "Description" ""
-			(at 0 0 90)
-			(unlocked yes)
-			(layer "F.Fab")
-			(hide yes)
-			(effects
-				(font
-					(size 1.27 1.27)
-					(thickness 0.15)
-				)
-			)
-		)
-		(attr smd)
-		(fp_line
-			(start -0.711252 -0.91)
-			(end 0.711252 -0.91)
-			(stroke
-				(width 0.12)
-				(type solid)
-			)
-			(layer "F.SilkS")
-		)
-		(fp_line
-			(start -0.711252 0.91)
-			(end 0.711252 0.91)
-			(stroke
-				(width 0.12)
-				(type solid)
-			)
-			(layer "F.SilkS")
-		)
-		(fp_line
-			(start 2.3 -1.15)
-			(end 2.3 1.15)
-			(stroke
-				(width 0.05)
-				(type solid)
-			)
-			(layer "F.CrtYd")
-		)
-		(fp_line
-			(start -2.3 -1.15)
-			(end 2.3 -1.15)
-			(stroke
-				(width 0.05)
-				(type solid)
-			)
-			(layer "F.CrtYd")
-		)
-		(fp_line
-			(start 2.3 1.15)
-			(end -2.3 1.15)
-			(stroke
-				(width 0.05)
-				(type solid)
-			)
-			(layer "F.CrtYd")
-		)
-		(fp_line
-			(start -2.3 1.15)
-			(end -2.3 -1.15)
-			(stroke
-				(width 0.05)
-				(type solid)
-			)
-			(layer "F.CrtYd")
-		)
-		(fp_line
-			(start 1.6 -0.8)
-			(end 1.6 0.8)
-			(stroke
-				(width 0.1)
-				(type solid)
-			)
-			(layer "F.Fab")
-		)
-		(fp_line
-			(start -1.6 -0.8)
-			(end 1.6 -0.8)
-			(stroke
-				(width 0.1)
-				(type solid)
-			)
-			(layer "F.Fab")
-		)
-		(fp_line
-			(start 1.6 0.8)
-			(end -1.6 0.8)
-			(stroke
-				(width 0.1)
-				(type solid)
-			)
-			(layer "F.Fab")
-		)
-		(fp_line
-			(start -1.6 0.8)
-			(end -1.6 -0.8)
-			(stroke
-				(width 0.1)
-				(type solid)
-			)
-			(layer "F.Fab")
-		)
-		(fp_text user "${REFERENCE}"
-			(at 0 0 90)
-			(layer "F.Fab")
-			(effects
-				(font
-					(size 0.8 0.8)
-					(thickness 0.12)
-				)
-			)
-		)
-		(pad "1" smd roundrect
-			(at -1.475 0 90)
-			(size 1.15 1.8)
-			(layers "F.Cu" "F.Paste" "F.Mask")
-			(roundrect_rratio 0.217391)
-			(net 3 "+5V")
-		)
-		(pad "2" smd roundrect
-			(at 1.475 0 90)
-			(size 1.15 1.8)
-			(layers "F.Cu" "F.Paste" "F.Mask")
-			(roundrect_rratio 0.217391)
-			(net 2 "GND")
-		)
-		(model "${KICAD8_3DMODEL_DIR}/Capacitor_SMD.3dshapes/C_1206_3216Metric.wrl"
-			(offset
-				(xyz 0 0 0)

Commit message: Add files via upload
Parts:
- C1, C2: value 12pF -> 18pF

Commit message: Add files via upload
Parts:
- added REF**: OSHW-Logo2_7.3x6mm_SilkScreen, Symbol:OSHW-Logo2_7.3x6mm_SilkScreen, B.Cu at (164.5, 88.4)

Commit message: Add files via upload
Other:
- board text added: "A2Pico2 v1.2 (c) 2026 Designed by Ralle Palaveev https://apple2.co.uk/ Concept by Oliver Schmidt https://a2retro.de/"
- board text removed: "A2Pico2 v1.2 (c) 2026 Designed by Ralle Palaveev https://apple2.co.uk/ Consept by Oliver Schmidt https://a2retro.de/"
Changed lines of the file:
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@@
 		)
 	)
-	(gr_text "A2Pico2 v1.2 (c) 2026\nDesigned by Ralle Palaveev https://apple2.co.uk/\nConsept by Oliver Schmidt https://a2retro.de/\n"
+	(gr_text "A2Pico2 v1.2 (c) 2026\nDesigned by Ralle Palaveev https://apple2.co.uk/\nConcept by Oliver Schmidt https://a2retro.de/\n"
 		(at 180.1368 100.6094 0)
 		(layer "B.SilkS")
@@
 	)
 	(gr_text "BOOTSEL"
-		(at 177.0302 83.625 0)
+		(at 176.7078 83.9978 0)
 		(layer "F.SilkS")
 		(effects

Commit message: Add files via upload
Routing:
- net LED: track 8.00 -> 12.6 mm, vias 2 -> 0
Changed lines of the file:
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@@
 	)
 	(via
-		(at 143.020482 87.4976)
+		(at 143.09 86.65)
 		(size 0.6)
 		(drill 0.3)
@@
 	)
 	(segment
-		(start 141.3764 87.9094)
-		(end 141.500664 87.785136)
+		(start 142.847704 87.53)
+		(end 144.16 87.53)
 		(width 0.15)
 		(layer "F.Cu")
@@
 	)
 	(segment
-		(start 141.500664 87.7268)
-		(end 141.56771 87.659754)
+		(start 144.85 86.84)
+		(end 144.85 85.01)
 		(width 0.15)
 		(layer "F.Cu")
@@
 	)
 	(segment
-		(start 141.56771 87.659754)
-		(end 142.26795 87.659754)
+		(start 138.564138 83.81)
+		(end 137.871338 83.1172)
 		(width 0.15)
 		(layer "F.Cu")
@@
 	)
 	(segment
-		(start 138.0574 83.1172)
-		(end 137.871338 83.1172)
+		(start 142.26795 87.659754)
+		(end 142.71795 87.659754)
 		(width 0.15)
 		(layer "F.Cu")
@@
 	)
 	(segment
-		(start 141.500664 87.785136)
-		(end 141.500664 87.7268)
+		(start 144.85 85.01)
+		(end 143.65 83.81)
 		(width 0.15)
 		(layer "F.Cu")
@@
 	)
 	(segment
-		(start 137.871338 83.1172)
-		(end 137.903482 83.1172)
+		(start 144.16 87.53)
+		(end 144.85 86.84)
 		(width 0.15)
 		(layer "F.Cu")
@@
 	)
 	(segment
-		(start 137.96795 83.213812)
-		(end 137.871338 83.1172)
+		(start 137.871338 83.1172)
+		(end 137.903482 83.1172)
 		(width 0.15)
 		(layer "F.Cu")
@@
 	)
 	(segment
-		(start 138.4046 83.4644)
-		(end 138.0574 83.1172)
+		(start 143.65 83.81)
+		(end 138.564138 83.81)
 		(width 0.15)
 		(layer "F.Cu")
 		(net 57)
 	)
-	(via
-		(at 138.4046 83.4644)
-		(size 0.5)
-		(drill 0.25)
-		(layers "F.Cu" "B.Cu")
-		(net 57)
-	)
-	(via
-		(at 141.3764 87.9094)
-		(size 0.5)
-		(drill 0.25)
-		(layers "F.Cu" "B.Cu")
-		(net 57)
-	)
-	(segment
-		(start 138.936529 83.4644)
-		(end 138.4046 83.4644)
-		(width 0.15)
-		(layer "In2.Cu")
-		(net 57)
-	)
-	(segment
-		(start 141.430507 85.958378)
-		(end 138.936529 83.4644)
-		(width 0.15)
-		(layer "In2.Cu")
-		(net 57)
-	)
 	(segment
-		(start 141.3764 87.9094)
-		(end 141.430507 87.855293)
+		(start 142.71795 87.659754)
+		(end 142.847704 87.53)
 		(width 0.15)
-		(layer "In2.Cu")
-		(net 57)
-	)
-	(segment
-		(start 141.430507 87.855293)
-		(end 141.430507 85.958378)
-		(width 0.15)
-		(layer "In2.Cu")
+		(layer "F.Cu")
 		(net 57)
 	)

Commit message: Add files via upload
Other:
- board text added: "A2Pico2.v1.2 (c) 2026 by Ralle Palaveev, https://apple2.co.uk/"
- board text removed: "A2PICO2.v1.2 (c) 2026 by Ralle Palaveev, https://apple2.co.uk/"
Changed lines of the file:
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@@
 		)
 		(fp_line
-			(start 8.8 7.42)
-			(end -9.32 7.42)
+			(start 8.35 7.42)
+			(end -8.45 7.42)
 			(stroke
 				(width 0.05)
@@
 		)
 		(fp_line
-			(start 8.8 -8.82)
-			(end 8.8 7.42)
+			(start 8.35 -8.82)
+			(end 8.35 7.42)
 			(stroke
 				(width 0.05)
@@
 		)
 		(fp_line
-			(start -9.32 7.42)
-			(end -9.32 -8.82)
+			(start -8.45 7.42)
+			(end -8.45 -8.82)
 			(stroke
 				(width 0.05)
@@
 		)
 		(fp_line
-			(start -9.32 -8.82)
-			(end 8.8 -8.82)
+			(start -8.45 -8.82)
+			(end 8.35 -8.82)
 			(stroke
 				(width 0.05)
@@
 		)
 	)
-	(gr_text "A2PICO2.v1.2 (c) 2026 by Ralle Palaveev, https://apple2.co.uk/"
+	(gr_text "A2Pico2.v1.2 (c) 2026 by Ralle Palaveev, https://apple2.co.uk/"
 		(at 148.3868 109.6518 0)
 		(layer "F.SilkS")
