File: v1.2/A2PICO2.v1.2.kicad_sch (KiCad schematic)
At the start: 63 parts, among them SW1 SW_BOOTSEL, SW2 SW_BOOTSEL, U1 RP2354B, U2 74LVC1G11, U3 ME6211, Y1 CM4012M00012001

Commit message: Add files via upload
Parts:
- removed C24: 100uF, Capacitor_SMD:C_0603_1608Metric, symbol Device:C_Small
Changed lines of the file:
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@@
 	)
 	(junction
-		(at 248.92 107.95)
-		(diameter 0)
-		(color 0 0 0 0)
-	)
-	(junction
 		(at 78.74 43.18)
 		(diameter 0)
@@
 	(wire
 		(pts
-			(xy 259.08 109.22) (xy 259.08 107.95)
-		)
-		(stroke
-			(width 0)
-			(type default)
-		)
-	)
-	(wire
-		(pts
 			(xy 248.92 109.22) (xy 248.92 107.95)
 		)
@@
 	(wire
 		(pts
-			(xy 259.08 107.95) (xy 248.92 107.95)
-		)
-		(stroke
-			(width 0)
-			(type default)
-		)
-	)
-	(wire
-		(pts
 			(xy 77.47 101.6) (xy 81.28 101.6)
 		)
@@
 	(symbol
 		(lib_id "power:GND")
-		(at 259.08 114.3 0)
-		(mirror y)
-		(unit 1)
-		(exclude_from_sim no)
-		(in_bom yes)
-		(on_board yes)
-		(dnp no)
-		(property "Reference" "#PWR046"
-			(at 259.08 120.65 0)
-			(effects
-				(font
-					(size 1.27 1.27)
-				)
-				(hide yes)
-			)
-		)
-		(property "Value" "GND"
-			(at 259.08 118.11 0)
-			(effects
-				(font
-					(size 1.27 1.27)
-				)
-			)
-		)
-		(property "Footprint" ""
-			(at 259.08 114.3 0)
-			(effects
-				(font
-					(size 1.27 1.27)
-				)
-				(hide yes)
-			)
-		)
-		(property "Datasheet" ""
-			(at 259.08 114.3 0)
-			(effects
-				(font
-					(size 1.27 1.27)
-				)
-				(hide yes)
-			)
-		)
-		(property "Description" ""
-			(at 259.08 114.3 0)
-			(effects
-				(font
-					(size 1.27 1.27)
-				)
-				(hide yes)
-			)
-		)
-		(pin "1"
-		)
-		(instances
-			(project "A2PICO2.v1.1"
-				(path "/019f2816-6bfb-4531-95b3-45f73cf5fc4b"
-					(reference "#PWR046")
-					(unit 1)
-				)
-			)
-		)
-	)
-	(symbol
-		(lib_id "power:GND")
 		(at 34.29 55.88 270)
 		(unit 1)
@@
 					(unit 1)
 				)
-			)
-		)
-	)
-	(symbol
-		(lib_id "Device:C_Small")
-		(at 259.08 111.76 0)
-		(unit 1)
-		(exclude_from_sim no)
-		(in_bom yes)
-		(on_board yes)
-		(dnp no)
-		(property "Reference" "C24"
-			(at 263.906 114.046 0)
-			(effects
-				(font
-					(size 1.27 1.27)
-				)
-				(justify right)
-			)
-		)
-		(property "Value" "100uF"
-			(at 260.35 109.474 0)
-			(effects
-				(font
-					(size 1.27 1.27)
-				)
-				(justify left)
-			)
-		)
-		(property "Footprint" "Capacitor_SMD:C_0603_1608Metric"
-			(at 259.08 111.76 0)
-			(effects
-				(font
-					(size 1.27 1.27)
-				)
-				(hide yes)
-			)
-		)
-		(property "Datasheet" "~"
-			(at 259.08 111.76 0)
-			(effects
-				(font
-					(size 1.27 1.27)
-				)
-				(hide yes)
-			)
-		)
-		(property "Description" ""
-			(at 259.08 111.76 0)
-			(effects
-				(font
-					(size 1.27 1.27)
-				)
-				(hide yes)
-			)
-		)
-		(property "Digikey" ""
-			(at 259.08 111.76 0)
-			(effects
-				(font
-					(size 1.27 1.27)
-				)
-				(hide yes)
-			)
-		)
-		(pin "1"
-		)
-		(pin "2"
-		)
-		(instances
-			(project "A2PICO2.v1.1"
-				(path "/019f2816-6bfb-4531-95b3-45f73cf5fc4b"
-					(reference "C24")
-					(unit 1)
-				)

Commit message: Add files via upload
Parts:
- C1, C2: value 12pF -> 18pF
Changed lines of the file:
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@@
 			)
 		)
-		(property "Value" "12pF"
+		(property "Value" "18pF"
 			(at 35.56 138.43 90)
 			(effects
@@
 			)
 		)
-		(property "Value" "12pF"
+		(property "Value" "18pF"
 			(at 35.56 128.27 90)
 			(effects
